File: hardware/Calunium_v2_smd_1.sch (EAGLE design)
At the start: 65 parts, among them IC1 MCP1702-3.3, IC2 DS1338, IC3 MCP1702-5.0, IC4 ATMEGA1284, IC5 MCP2200, Q1 2N7002, X1 PWR, X2 JTAG, X3 USB, X6 MICRO-SD-SOCKETHIROSE-DM3D, Y1 32k768, Y2 16MHz, Y3 12MHz

Commit message: Misc changes
Parts:
- removed IC3: MCP1702-5.0, SteveMarple:MCP1702
- removed JP4: USB PWR, SparkFun:JUMPER-2PTH
- removed JP6: VREG PWR, SparkFun:JUMPER-2PTH
- added IC6: TSR 1-2450, SteveMarple:V_REG_78XXTSR-1-XXXX
- added JP9: USB/VIN, SparkFun:JUMPER-3PTH
- C2: value 1u -> 10u; device SteveMarple:C-EU1206-HAND -> SteveMarple:CAP_POLPTH2
- IC1: value MCP1702-3.3 -> LD1117S33TR; device SteveMarple:MCP1702 -> SteveMarple:V_REG_LD1117VXXSOT223-HAND
- R1, R2: value 1k -> 560R
Connections:
- net +3V3: now also C2.+, IC1.OUT; no longer C2.1, IC1.VOUT
- net +5V: now also IC1.IN, JP9.2; no longer IC1.VIN, JP4.2, JP6.2
- net +5V_USB: now also JP9.3; no longer JP4.1
- net GND: now also C2.-, IC6.GND; no longer C2.2, IC3.GND
- net N$14: now also IC6.OUT, JP9.1; no longer IC3.VOUT, JP6.1
- net VIN: now also IC6.IN; no longer IC3.VIN
