File: hardware/PoE_mag_main.brd (EAGLE design)
At the start: 0 parts

Commit message: Misc changes
Parts:
- added BAT1: CR2032, SparkFun:BATTCOM_20MM_PTH
- added C1, C2, C8: 1u, SteveMarple:1206-HAND
- added C10, C11, C15, C16: 22p, SteveMarple:0805-HAND
- added C12, C14, C19, C20, C3, C5, C7, C9: 100n, SteveMarple:1206-HAND
- added C13: 10n, SteveMarple:1206-HAND
- added C17, C18: 15p, SteveMarple:0805-HAND
- added C4: 100p, SteveMarple:1206-HAND
- added C6: 4u7, SparkFun:CPOL-RADIAL-10UF-25V
- added D1, D2: BAT85, SteveMarple:SOT23-3-HAND
- added H1, H2, H3, H4: (no value), holes:3,0-PAD
- added IC1: MCP1702-3.3, SteveMarple:TO-92
- added IC2: DS1338, SteveMarple:SO08
- added IC3: MCP1702-5.0, SteveMarple:TO-92
- added IC4: ATMEGA1284, SteveMarple:DIL40
- added IC5: MCP2200, SteveMarple:SO20
- added JP1: SQW D6/D15, SparkFun:1X03
- added JP2: SDA/A4, SparkFun:1X03
- added JP3: SCL/A5, SparkFun:1X03
- added JP4: USB PWR, SparkFun:1X02
- added JP5: 3V3/5V, SparkFun:1X03
- added JP6: VREG PWR, SparkFun:1X02
- added JP7: AUTO RST, SparkFun:1X02
- added JP8: ISP VCC, SparkFun:1X02
- added L1: 10uH, SteveMarple:1210-HAND
- added L2: FERRITE, SteveMarple:0805-HAND
- added LED1: D13, SparkFun:LED3MM
- added LED2: PWR, SparkFun:LED3MM
- added Q1: 2N7002, SteveMarple:SOT23-3-ROTATED
- added R1, R2, R7, R9: 1k, SteveMarple:1206-HAND
- added R10: 1M, SteveMarple:1206-HAND
- added R3, R6: 10k, SteveMarple:1206-HAND
- added R4, R5: 4k7, SteveMarple:1206-HAND
- added R8: 0R, SteveMarple:1206-HAND
- added S1: RESET, SparkFun:TACTILE-PTH
- added SENS1: LM61, SteveMarple:TO-92
- added U$1: CALUNIUM-SHIELD-V3V3-NO-HOLES-NO-TEXT, SteveMarple:CALUNIUM-SHIELD-NO-OUTLINE-NO-HOLES-NO-TEXT-V3
- added X1: PWR, con-molex:22-23-2071
- added X2: JTAG, SteveMarple:CON-HARTING-ML10
- added X3: USB, SteveMarple:USB-B-PTH
- added X6: MICRO-SD-SOCKETHIROSE-DM3D, SteveMarple:MICRO-SD-SOCKET-HIROSE-DM3D
- added Y1: 32k768, SteveMarple:TC38H
- added Y2: 16MHz, SteveMarple:HC49U-V-RESONATOR
- added Y3: 12MHz, SteveMarple:HC49U-V-RESONATOR
Connections:
- new net !MCP2200_RESET: IC5.4, R9.1
- new net !RESET: C12.2, D1.1, IC4.9, R6.1, S1.3, S1.4, U$1.!ISP_RESET, U$1.!RESET@0, X2.6
- new net +3V3: C19.1, C2.1, IC1.3, IC5.17, JP5.1, U$1.3.3V, X1.3
- new net +5V: C1.1, IC1.2, JP4.2, JP5.3, JP6.2, U$1.5V, X1.4
- new net +5V_USB: C13.1, JP4.1, L2.2, X1.1
- new net 0(RX0): IC4.14, IC5.10, U$1.0(RX0)
- new net 1(TX0): IC4.15, IC5.12, U$1.1(TX0)
- new net 10: IC4.5, U$1.10
- new net 11(MOSI): IC4.6, U$1.11@0, U$1.ISP_MOSI, X6.CMD
- new net 12(MISO): IC4.7, U$1.12@0, U$1.ISP_MISO, X6.DAT0
- new net 13(SCK): IC4.8, Q1.1, R10.2, U$1.13@0, U$1.ISP_SCK, X6.CLK
- new net 14: IC4.29, U$1.14
- new net 15: IC4.28, JP1.1, U$1.15
- new net 16(TDI): IC4.27, U$1.16, X2.9
- new net 17(TDO): IC4.26, U$1.17, X2.3
- new net 18(TMS): IC4.25, U$1.18, X2.5
- new net 19(TCK): IC4.24, U$1.19, X2.1
- new net 2(RX1): IC4.16, U$1.2@0, U$1.2@1
- new net 20(SDA): IC2.5, IC4.23, JP2.3, R5.1, U$1.20@0, U$1.20@1, U$1.SDA
- new net 21(SCL): IC2.6, IC4.22, JP3.3, R4.1, U$1.21@0, U$1.21@1, U$1.SCL
- new net 22: IC4.18, U$1.22, X6.CD/DAT3
- new net 23: IC4.21, U$1.23
- new net 3(TX1): IC4.17, U$1.3@0, U$1.3@1
- new net 4: IC4.1, U$1.4
- new net 5: IC4.2, U$1.5
- new net 6: IC4.3, JP1.3, U$1.6
- new net 7: IC4.4, U$1.7
- new net 8: IC4.20, U$1.8
- new net 9: IC4.19, U$1.9
- new net A0: IC4.33, U$1.A0
- new net A1: IC4.34, U$1.A1
- new net A2: IC4.35, U$1.A2
- new net A3: IC4.36, U$1.A3
- new net A4: IC4.37, JP2.1
- new net A4/SDA: JP2.2, U$1.A4/SDA
- new net A5: IC4.38, JP3.1
- new net A5/SCL: JP3.2, U$1.A5/SCL
- new net A6: IC4.39, SENS1.1, U$1.A6
- new net A7: IC4.40, SENS1.2, U$1.A7
- new net AREF: C5.1, IC4.32, U$1.AREF
- new net AUTO_RESET: IC5.11, JP7.1
- new net AVCC: C9.1, IC4.30, L1.1
- new net GND: BAT1.2, C1.2, C10.2, C11.2, C13.2, C14.2, C15.2, C16.2, C17.2, C18.2, C19.2, C2.2, C20.2, C3.2, C4.2, C5.2, C6.2, C7.2, C8.2, C9.2, H1.B3,0, H2.B3,0, H3.B3,0, H4.B3,0, IC1.1, IC2.4, IC3.1, IC4.11, IC4.31, IC5.20, LED2.K, Q1.2, R10.1, S1.1, S1.2, SENS1.3, U$1.GND@0, U$1.GND@1, U$1.GND@2, U$1.GND@3, X1.5, X1.6, X2.10, X2.2, X3.GND, X6.GND, X6.SHIELD@0, Y2.GND, Y3.GND
- new net N$1: C11.1, IC4.13, Y2.2
- new net N$11: C4.1, IC2.3, R7.2, R8.2
- new net N$12: C17.1, IC2.2, Y1.1
- new net N$14: IC3.3, JP6.1
- new net N$15: C12.1, JP7.2
- new net N$16: L2.1, X3.VBUS
- new net N$18: C15.1, IC5.2, Y3.1
- new net N$2: C10.1, IC4.12, Y2.1
- new net N$3: LED1.A, R1.1
- new net N$4: LED1.K, Q1.3
- new net N$5: C18.1, IC2.1, Y1.2
- new net N$6: JP8.1, U$1.ISP_VCC
- new net N$7: C16.1, IC5.3, Y3.2
- new net N$8: LED2.A, R2.1
- new net N$9: D2.3, R7.1
- new net SQW: IC2.7, JP1.2, R3.1
- new net USB_D+: IC5.19, X3.D+
- new net USB_D-: IC5.18, X3.D-
- new net VBATT: BAT1.1, D2.1, R8.1, X1.2
- new net VCC: C14.1, C20.1, C3.1, C6.1, C7.1, D1.3, IC2.8, IC4.10, IC5.1, JP5.2, JP8.2, L1.2, R1.2, R2.2, R3.2, R4.2, R5.2, R6.2, R9.2, U$1.IOREF, X2.4, X6.VDD
- new net VIN: C8.1, IC3.2, U$1.VIN, X1.7
Routing:
- net N$7: track 0.00 -> 19.1 mm
- net USB_D+: track 0.00 -> 16.1 mm, vias 0 -> 1
- net USB_D-: track 0.00 -> 15.9 mm, vias 0 -> 1
- net N$18: track 0.00 -> 14.8 mm
- net AVCC: track 0.00 -> 9.53 mm
- net N$2: track 0.00 -> 8.04 mm
- net N$1: track 0.00 -> 8.04 mm
- net N$5: track 0.00 -> 7.51 mm
- net N$12: track 0.00 -> 6.99 mm
- net VCC: track 0.00 -> 4.86 mm
- net AREF: track 0.00 -> 4.45 mm
Other:
- board outline added: 158.8 x 99.1 mm
- board text added: "!RESET"
- board text added: "-ShareAlike 3.0 Unported License"
- board text added: "0"
- board text added: "1"
- board text added: "10"
- board text added: "11"
- board text added: "12"
- board text added: "13"
- board text added: "14"
- board text added: "15"
- board text added: "16"
- board text added: "17"
- board text added: "18"
- board text added: "19"
- board text added: "2"
- board text added: "20"
- board text added: "21"
- board text added: "22"
- board text added: "23"
- board text added: "3"
- board text added: "3V3"
- board text added: "4"
- board text added: "5"
- board text added: "5V"
- board text added: "6"
- board text added: "7"
- board text added: "8"
- board text added: "9"
- board text added: ">DRAWING_NAME"
- board text added: ">PLOT_DATE_TIME"
- board text added: "A0"
- board text added: "A1"
- board text added: "A2"
- board text added: "A3"
- board text added: "A4"
- board text added: "A5"
- board text added: "A6"
- board text added: "A7"
- board text added: "AREF"
- board text added: "Calunium v2.1a"
- board text added: "Copyright Steve Marple 2012"
- board text added: "GND"
- board text added: "IOREF"
- board text added: "License: Creative Commons Attribution"
- board text added: "MHz"
- board text added: "NC"
- board text added: "RESET"
- board text added: "RX0"
- board text added: "RX1"
- board text added: "S/N"
- board text added: "SCL"
- board text added: "SDA"
- board text added: "TX0"
- board text added: "TX1"
- board text added: "Vin"
- board text added: "calunium@stevemarple.co.uk"
- board text added: "https://github.com/stevemarple/Calunium"
