File: hardware/PoE_mag_main.sch (EAGLE design)
At the start: 0 parts

Commit message: Misc changes
Parts:
- added BAT1: CR2032, SparkFun:BATTERY20PTH
- added C1, C2, C8: 1u, SteveMarple:C-EU1206-HAND
- added C10, C11, C15, C16: 22p, SteveMarple:C-EU0805-HAND
- added C12, C14, C19, C20, C3, C5, C7, C9: 100n, SteveMarple:C-EU1206-HAND
- added C13: 10n, SteveMarple:C-EU1206-HAND
- added C17, C18: 15p, SteveMarple:C-EU0805-HAND
- added C4: 100p, SteveMarple:C-EU1206-HAND
- added C6: 4u7, SparkFun:CAP_POLPTH2
- added D1, D2: BAT85, SteveMarple:DIODE-SCHOTTKYSOT23-1-3-HAND
- added H1, H2, H3, H4: MOUNT-PAD-ROUND3.0, holes:MOUNT-PAD-ROUND3.0
- added IC1: MCP1702-3.3, SteveMarple:MCP1702
- added IC2: DS1338, SteveMarple:DS1307SO08
- added IC3: MCP1702-5.0, SteveMarple:MCP1702
- added IC4: ATMEGA1284, SteveMarple:ATMEGA644-20PU
- added IC5: MCP2200, SteveMarple:MCP2200
- added JP1: SQW D6/D15, SparkFun:JUMPER-3PTH
- added JP2: SDA/A4, SparkFun:JUMPER-3PTH
- added JP3: SCL/A5, SparkFun:JUMPER-3PTH
- added JP4: USB PWR, SparkFun:JUMPER-2PTH
- added JP5: 3V3/5V, SparkFun:JUMPER-3PTH
- added JP6: VREG PWR, SparkFun:JUMPER-2PTH
- added JP7: AUTO RST, SparkFun:JUMPER-2PTH
- added JP8: ISP VCC, SparkFun:JUMPER-2PTH
- added L1: 10uH, SteveMarple:INDUCTOR1210-HAND
- added L2: FERRITE, SteveMarple:INDUCTOR0805-HAND
- added LED1: D13, SparkFun:LED3MM
- added LED2: PWR, SparkFun:LED3MM
- added Q1: 2N7002, SteveMarple:2N7002
- added R1, R2, R7, R9: 1k, SteveMarple:RESISTOR1206-HAND
- added R10: 1M, SteveMarple:RESISTOR1206-HAND
- added R3, R6: 10k, SteveMarple:RESISTOR1206-HAND
- added R4, R5: 4k7, SteveMarple:RESISTOR1206-HAND
- added R8: 0R, SteveMarple:RESISTOR1206-HAND
- added S1: RESET, SparkFun:TAC_SWITCHPTH
- added SENS1: LM61, SteveMarple:LM61
- added U$1: CALUNIUM-SHIELD-V3V3-NO-HOLES-NO-TEXT, SteveMarple:CALUNIUM-SHIELD-V3V3-NO-HOLES-NO-TEXT
- added X1: PWR, con-molex:22-23-2071
- added X2: JTAG, SteveMarple:ATMEL-JTAG
- added X3: USB, SteveMarple:USBPTH
- added X6: MICRO-SD-SOCKETHIROSE-DM3D, SteveMarple:MICRO-SD-SOCKETHIROSE-DM3D
- added Y1: 32k768, SteveMarple:CRYSTALTC38H
- added Y2: 16MHz, SteveMarple:CRYSTAL-RESONATOR
- added Y3: 12MHz, SteveMarple:CRYSTAL-RESONATOR
Connections:
- new net !MCP2200_RESET: IC5.!RST, R9.1
- new net !RESET: C12.2, D1.A, IC4.!RESET, R6.1, S1.3, S1.4, U$1.!RESET@0, U$1.!RESET@1, X2.!SRST
- new net +3V3: C19.1, C2.1, IC1.VOUT, IC5.VUSB, JP5.1, U$1.3.3V, X1-3.S
- new net +5V: C1.1, IC1.VIN, JP4.2, JP5.3, JP6.2, U$1.5V, X1-4.S
- new net +5V_USB: C13.1, JP4.1, L2.2, X1-1.S
- new net 0(RX0): IC4.PCINT24/RXD0_PD0, IC5.TX, U$1.0(RX0)
- new net 1(TX0): IC4.PCINT25/TXD0_PD1, IC5.RX, U$1.1(TX0)
- new net 10: IC4.PCINT12/OC0B/SS_PB4, U$1.10
- new net 11(MOSI): IC4.PCINT13/MOSI_PB5, U$1.11(MOSI), U$1.ISP_MOSI, X6.CMD
- new net 12(MISO): IC4.PCINT14/MISO_PB6, U$1.12(MISO), U$1.ISP_MISO, X6.DAT0
- new net 13(SCK): IC4.PCINT15/SCK_PB7, Q1.G, R10.2, U$1.13(SCK), U$1.ISP_SCK, X6.CLK
- new net 14: IC4.PCINT23/TOSC2_PC7, U$1.14
- new net 15: IC4.PCINT22/TOSC1_PC6, JP1.1, U$1.15
- new net 16(TDI): IC4.PCINT21/TDI_PC5, U$1.16, X2.TDI
- new net 17(TDO): IC4.PCINT20/TDO_PC4, U$1.17, X2.TDO
- new net 18(TMS): IC4.PCINT19/TMS_PC3, U$1.18, X2.TMS
- new net 19(TCK): IC4.PCINT18/TCK_PC2, U$1.19, X2.TCK
- new net 2(RX1): IC4.PCINT26/INT0_PD2, U$1.2(RX1)@0, U$1.2(RX1)@1
- new net 20(SDA): IC2.SDA, IC4.PCINT17/SDA_PC1, JP2.3, R5.1, U$1.20(SDA)@0, U$1.20(SDA)@1, U$1.SDA
- new net 21(SCL): IC2.SCL, IC4.PCINT16/SCL_PC0, JP3.3, R4.1, U$1.21(SCL)@0, U$1.21(SCL)@1, U$1.SCL
- new net 22: IC4.PCINT28/OC1B_PD4, U$1.22, X6.CD/DAT3
- new net 23: IC4.PCINT31/OC2A_PD7, U$1.23
- new net 3(TX1): IC4.PCINT27/INT1_PD3, U$1.3(TX1)@0, U$1.3(TX1)@1
- new net 4: IC4.PCINT8/XCK0/T0_PB0, U$1.4
- new net 5: IC4.PCINT9/CLKO/T1_PB1, U$1.5
- new net 6: IC4.PCINT10/INT2/AIN0_PB2, JP1.3, U$1.6
- new net 7: IC4.PCINT11/OC0A/AIN1_PB3, U$1.7
- new net 8: IC4.PCINT30/OC2B/ICP_PD6, U$1.8
- new net 9: IC4.PCINT29/OC1A_PD5, U$1.9
- new net A0: IC4.PCINT7/ADC7_PA7, U$1.A0
- new net A1: IC4.PCINT6/ADC6_PA6, U$1.A1
- new net A2: IC4.PCINT5/ADC5_PA5, U$1.A2
- new net A3: IC4.PCINT4/ADC4_PA4, U$1.A3
- new net A4: IC4.PCINT3/ADC3_PA3, JP2.1
- new net A4/SDA: JP2.2, U$1.A4
- new net A5: IC4.PCINT2/ADC2_PA2, JP3.1
- new net A5/SCL: JP3.2, U$1.A5
- new net A6: IC4.PCINT1/ADC1_PA1, SENS1.VS, U$1.A6
- new net A7: IC4.PCINT0/ADC0_PA0, SENS1.VOUT, U$1.A7
- new net AREF: C5.1, IC4.AREF, U$1.AREF
- new net AUTO_RESET: IC5.!RTS, JP7.1
- new net AVCC: C9.1, IC4.AVCC, L1.1
- new net GND: BAT1.-, C1.2, C10.2, C11.2, C13.2, C14.2, C15.2, C16.2, C17.2, C18.2, C19.2, C2.2, C20.2, C3.2, C4.2, C5.2, C6.-, C7.2, C8.2, C9.2, H1.MOUNT, H2.MOUNT, H3.MOUNT, H4.MOUNT, IC1.GND, IC2.GND, IC3.GND, IC4.GND, IC4.GND@1, IC5.VSS, LED2.C, Q1.S, R10.1, S1.1, S1.2, SENS1.GND, U$1.GND, X1-5.S, X1-6.S, X2.GND@0, X2.GND@1, X3.GND, X6.SHIELD, X6.VSS, Y2.2, Y3.2
- new net N$1: C11.1, IC4.XTAL1, Y2.3
- new net N$11: C4.1, IC2.VBATT, R7.2, R8.2
- new net N$12: C17.1, IC2.X2, Y1.1
- new net N$14: IC3.VOUT, JP6.1
- new net N$15: C12.1, JP7.2
- new net N$16: L2.1, X3.VBUS
- new net N$18: C15.1, IC5.OSC1, Y3.1
- new net N$2: C10.1, IC4.XTAL2, Y2.1
- new net N$3: LED1.A, R1.1
- new net N$4: LED1.C, Q1.D
- new net N$5: C18.1, IC2.X1, Y1.2
- new net N$6: JP8.1, U$1.ISP_VCC
- new net N$7: C16.1, IC5.OSC2, Y3.3
- new net N$8: LED2.A, R2.1
- new net N$9: D2.C, R7.1
- new net SQW: IC2.SQW, JP1.2, R3.1
- new net USB_D+: IC5.D+, X3.D+
- new net USB_D-: IC5.D-, X3.D-
- new net VBATT: BAT1.+, D2.A, R8.1, X1-2.S
- new net VCC: C14.1, C20.1, C3.1, C6.+, C7.1, D1.C, IC2.VCC, IC4.VCC, IC5.VDD, JP5.2, JP8.2, L1.2, R1.2, R2.2, R3.2, R4.2, R5.2, R6.2, R9.2, U$1.IOREF, X2.VTREF, X6.VDD
- new net VIN: C8.1, IC3.VIN, U$1.VIN, X1-7.S
Other:
- note added: "2.1a"
- note added: "3V3 regulator"
- note added: "5V regulator"
- note added: "ATmega324/644/1284"
- note added: "Add FET to switch fan"
- note added: "D13 LED"
- note added: "JTAG header"
- note added: "MicroSD socket"
- note added: "Omit load capacitors if resonator"
- note added: "Onboard peripherals"
- note added: "Power LED"
- note added: "Power and connectors"
- note added: "Power header"
- note added: "Power selection"
- note added: "RTC battery"
- note added: "Real time clock"
- note added: "Reset"
- note added: "Steve Marple"
- note added: "TODO Swap MCP1702 (3V3 and 5V) for SMD"
- note added: "Temperature sensor"
- note added: "UART-USB converter"
- note added: "USB power and filtering"
- note added: "fitted instead of crystal"
