File: hardware/FLC100_level_shifting.brd (EAGLE design)
At the start: 99.1 x 53.3 mm, 30 parts, among them X1 RJ45, X2 RJ11, X3 CLOUD SENSOR, X5 HUMIDITY

Commit message: Layout fixes
Parts:
- removed C8: 100n, SteveMarple:1206-HAND
- removed C9: 100u, SteveMarple:CPOL-RADIAL-10UF-25V
- removed JP6: CLOUD CTRL, SparkFun:1X02
- removed R15, R16, R17, R18, R19, R20: 10k, SteveMarple:1206-HAND
- removed U$1, U$13, U$14, U$2, U$3: PAD, SteveMarple:PAD
- removed U$6, U$7: PCA9517ASOIC, SteveMarple:SO08
- removed X5: HUMIDITY, SteveMarple:ML8
- added C1, C2, C4, C5, C7: 100n, SteveMarple:1206-HAND
- added C6: 100u, SteveMarple:CPOL-RADIAL-10UF-25V
- added D1: BAS40, SteveMarple:SOT23-3-HAND
- added IC1, IC2: PCA9517A, SteveMarple:SO08
- added R10: 1k, SteveMarple:1206-HAND
- added R11, R12, R6, R7, R8: 10k, SteveMarple:1206-HAND
- added R9: 3k, SteveMarple:1206-HAND
- added X4: HUMIDITY, SteveMarple:ML8
- JP2: value VIN ADC -> MAG VCC; device SparkFun:1X02 -> SparkFun:1X03
- JP3: value MAG VCC -> CLOUD CTRL; device SparkFun:1X03 -> SparkFun:1X02
- R4: value 1k -> 10k; device SteveMarple:RES-AXIAL-0.4 -> SteveMarple:1206-HAND
- moved R5 98.0 mm to (44.5, 31.8), turned to 180 degrees
- moved R3 90.1 mm to (24.1, 43.2), turned to 180 degrees
- moved R2 75.1 mm to (24.1, 24.1), turned to 180 degrees
- moved C3 66.4 mm to (40.6, 40.6), turned to 180 degrees
- moved R1 61.0 mm to (24.1, 20.3), turned to 180 degrees
- moved JP2 59.3 mm to (12.7, 50.8), turned to 180 degrees
- moved JP3 56.6 mm to (54.6, 12.7), turned to 0 degrees
- moved JP1 38.9 mm to (20.3, 50.8), turned to 180 degrees
- moved U$5 36.4 mm to (62.2, 22.9)
- moved X3 29.6 mm to (55.9, 43.2)
- moved R4 20.6 mm to (24.1, 39.4), turned to 180 degrees
Connections:
- removed net N$6: R4.P$1, X1.3, X2.2
- removed net SHDN: R4.P$2
- net +3V3: now also C5.1, C6.1, JP2.3, X4.8; no longer C3.1, C9.1, JP3.3, U$3.1, X5.8
- net +5V: no longer U$2.1
- net 16: now also IC2.3, R5.1; no longer R2.1, U$7.3
- net 18: now also JP3.1; no longer JP6.1
- net 19: now also IC2.2, R6.1; no longer R1.1, U$7.2
- net 20(SDA): now also IC1.3, R1.1; no longer R18.1, U$6.3
- net 21(SCL): now also IC1.2, R2.1; no longer R17.1, U$6.2
- net A2: now also D1.1, R10.2, R9.2; no longer JP2.2
- net A4/SDA: now also R11.1, X4.7; no longer R15.1, X5.7
- net A5/SCL: now also R12.1, X4.5; no longer R16.1, X5.5
- net CLOUD_SCL: now also IC2.7, R8.1; no longer R5.1, U$7.7
- net CLOUD_SDA: now also IC2.6, R7.1; no longer R3.1, U$7.6
- net CLOUD_VCC: now also C4.1, IC2.5, IC2.8, R7.2, R8.2; no longer R3.2, R5.2, U$7.5, U$7.8
- net GND: now also C1.2, C2.2, C4.2, C5.2, C6.2, C7.2, IC1.4, IC2.4, R10.1, X1.3, X2.2, X4.4; no longer C8.2, C9.2, U$6.4, U$7.4, X5.4
- net MAG_SCL: now also IC1.7, R4.1; no longer R20.1, U$6.7
- net MAG_SDA: now also IC1.6, R3.1; no longer R19.1, U$6.6
- net MAG_VCC: now also C2.1, IC1.5, IC1.8, R3.2, R4.2; no longer R19.2, R20.2, U$6.5, U$6.8
- net N$16: now also U$5.1, X4.3; no longer U$13.1, X5.3
- net N$22: now also C7.1, R11.2, R12.2, X4.6; no longer C8.1, R15.2, R16.2, X5.6
- net N$3: now also JP3.2; no longer JP6.2
- net N$7: now also JP2.2; no longer JP3.2
- net VCC: now also C1.1, C3.1, D1.3, IC1.1, IC2.1, R5.2, R6.2, X4.1; no longer R17.2, R18.2, U$5.1, U$6.1, U$7.1, X5.1
- net VIN: now also R9.1, X4.2; no longer JP3.1, U$1.1, X5.2
Other:
- board outline removed
- board text removed: "+5V"
- board text removed: ">DRAWING_NAME"
- board text removed: ">PLOT_DATE_TIME"
- board text removed: "IOREF"
