File: hardware/FLC100_level_shifting.sch (EAGLE design)
At the start: 30 parts, among them X1 RJ45, X2 RJ11, X3 CLOUD SENSOR, X5 HUMIDITY

Commit message: Layout fixes
Parts:
- removed JP6: CLOUD CTRL, SparkFun:JUMPER-2PTH
- removed R17, R18, R19, R20: 10k, SteveMarple:RESISTOR1206-HAND
- removed U$1, U$13, U$14, U$2, U$3: PAD, SteveMarple:PAD
- removed U$6, U$7: PCA9517ASOIC, SteveMarple:PCA9517ASOIC
- added C1, C2, C4, C5: 100n, SteveMarple:C-EU1206-HAND
- added D1: BAS40, SteveMarple:DIODE-SCHOTTKYSOT23-1-3-HAND
- added IC1, IC2: PCA9517A, SteveMarple:PCA9517ASOIC
- added R10: 1k, SteveMarple:RESISTOR1206-HAND
- added R6, R7, R8: 10k, SteveMarple:RESISTOR1206-HAND
- added R9: 3k, SteveMarple:RESISTOR1206-HAND
- JP2: value VIN ADC -> MAG VCC; device SparkFun:JUMPER-2PTH -> SparkFun:JUMPER-3PTH
- JP3: value MAG VCC -> CLOUD CTRL; device SparkFun:JUMPER-3PTH -> SparkFun:JUMPER-2PTH
- R4: value 1k -> 10k; device SteveMarple:RESISTOR -> SteveMarple:RESISTOR1206-HAND
- renumbered C8 to C7, C9 to C6, R15 to R11, R16 to R12, X5 to X4
Connections:
- removed net N$6: R4.1, X1.3, X2.2
- removed net SHDN: R4.2
- net +3V3: now also C5.1, JP2.3; no longer C3.1, JP3.3, U$3.1
- net +5V: no longer U$2.1
- net 16: now also IC2.SDA_A, R5.1; no longer R2.1, U$7.SDA_A
- net 18: now also JP3.1; no longer JP6.1
- net 19: now also IC2.SCL_A, R6.1; no longer R1.1, U$7.SCL_A
- net 20(SDA): now also IC1.SDA_A, R1.1; no longer R18.1, U$6.SDA_A
- net 21(SCL): now also IC1.SCL_A, R2.1; no longer R17.1, U$6.SCL_A
- net A2: now also D1.A, R10.2, R9.2; no longer JP2.2
- net CLOUD_SCL: now also IC2.SCL_B, R8.1; no longer R5.1, U$7.SCL_B
- net CLOUD_SDA: now also IC2.SDA_B, R7.1; no longer R3.1, U$7.SDA_B
- net CLOUD_VCC: now also C4.1, IC2.EN, IC2.VCC_B, R7.2, R8.2; no longer R3.2, R5.2, U$7.EN, U$7.VCC_B
- net GND: now also C1.2, C2.2, C4.2, C5.2, IC1.GND, IC2.GND, R10.1, X1.3, X2.2; no longer U$6.GND, U$7.GND
- net MAG_SCL: now also IC1.SCL_B, R4.1; no longer R20.1, U$6.SCL_B
- net MAG_SDA: now also IC1.SDA_B, R3.1; no longer R19.1, U$6.SDA_B
- net MAG_VCC: now also C2.1, IC1.EN, IC1.VCC_B, R3.2, R4.2; no longer R19.2, R20.2, U$6.EN, U$6.VCC_B
- net N$16: now also U$5.1; no longer U$13.1
- net N$3: now also JP3.2; no longer JP6.2
- net N$7: now also JP2.2; no longer JP3.2
- net VCC: now also C1.1, C3.1, D1.C, IC1.VCC_A, IC2.VCC_A, R5.2, R6.2; no longer R17.2, R18.2, U$5.1, U$6.VCC_A, U$7.VCC_A
- net VIN: now also R9.1; no longer JP3.1, U$1.1
Other:
- note added: "SHUTDOWN held low permanently for PoE operation"
- moved on the sheet: C3, R1, R2, R3, R4, R5
