File: hardware/NV08C_GPS_shield_v1.1_reduced.brd (EAGLE design)
At the start: 99.1 x 53.3 mm, 36 parts, among them IC2 74LVC1T45SOT23-HAND, IC5 74LVC1T45SOT23-HAND, IC6 74LVC1T45SOT23-HAND, IC7 74LVC1T45SOT23-HAND, X2 CONN-SMATHD, X3 UFL

Commit message: Layout fixes
Parts:
- removed IC5, IC6, IC7: 74LVC1T45SOT23-HAND, SteveMarple:SOT23-6-HAND
- removed JP6: V ANT, SparkFun:1X03
- removed JP8: PPS 7/6, SparkFun:1X03
- removed R4: 100k, SteveMarple:1206-HAND
- removed R5: 10k, SteveMarple:1206-HAND
- removed X3: UFL, SteveMarple:CONN-UFL-HAND-SOLDERING
- added C1, C2: 100n, SteveMarple:1206-HAND
- added C14: 22p, SteveMarple:0805-HAND
- added C15: 1u, SteveMarple:1206-HAND
- added C16: 4u7, SteveMarple:CPOL-RADIAL-10UF-25V
- added IC1, IC3, IC4: 74LVC1T45SOT23-HAND, SteveMarple:SOT23-6-HAND
- added JP1: GPS !RESET! (A0), SparkFun:1X02
- added JP2: V ANT, SparkFun:1X03
- added R2: 100k, SteveMarple:1206-HAND
- added R3: 10k, SteveMarple:1206-HAND
- added X1: CONN-SMATHD, SteveMarple:SMA-THD
- C10: value 1u -> 22p; device SteveMarple:1206-HAND -> SteveMarple:0805-HAND
- C12, C9: value 22p -> 1u; device SteveMarple:0805-HAND -> SteveMarple:1206-HAND
- C7, C8: value 1u -> 100n
- JP4: value GPS !RESET! (A0) -> PPS 7/6; device SparkFun:1X02 -> SparkFun:1X03
- X2: value CONN-SMATHD -> UFL; device SteveMarple:SMA-THD -> SteveMarple:CONN-UFL-HAND-SOLDERING
- moved C8 37.6 mm to (61.0, 15.2)
- moved C12 37.2 mm to (53.3, 15.2), turned to 270 degrees
- moved JP4 33.1 mm to (87.6, 39.4), turned to 0 degrees
- moved C10 32.4 mm to (33.0, 37.8), turned to 180 degrees
- moved C7 23.7 mm to (68.6, 25.4)
- moved IC2 23.0 mm to (64.8, 30.5)
- moved C6 22.9 mm to (61.0, 35.6)
- moved DP1 19.4 mm to (40.6, 3.81), turned to 90 degrees
- moved C5 18.9 mm to (68.6, 45.7), turned to 0 degrees
- moved C3 12.8 mm to (61.0, 25.4)
- moved X2 9.52 mm to (12.7, 14.6), turned to 180 degrees
- moved C11 8.54 mm to (47.6, 8.89), turned to 0 degrees
- moved C13 6.98 mm to (16.5, 20.3), turned to 180 degrees
- moved C4 6.84 mm to (68.6, 15.2)
- moved R1 3.18 mm to (71.1, 10.2)
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- renumbered JP7 to JP3, U$16 to U$1, U$18 to U$2, U$19 to U$3, U$20 to U$4, U$21 to U$5, U$22 to U$6, U$23 to U$7, U$24 to U$8, U$25 to U$9
Connections:
- removed net IOREF: C3.1, C4.1, IC2.6, IC5.6, IC6.1, IC7.1, R1.2, R4.2
- new net VCC: C1.1, C2.1, C3.1, C4.1, IC1.6, IC2.6, IC3.1, IC4.1, R1.2, R2.2
- net !GPS_RESET: now also IC1.3; no longer IC2.3
- net +3V3: now also C12.1, C7.1, IC1.1, IC3.6, IC4.6, JP2.3; no longer IC5.1, IC6.6, IC7.6, JP6.3
- net +5V: now also JP2.1; no longer C7.1, JP6.1
- net 2(RX1): now also R3.1; no longer R5.1
- net 3(TX1): now also IC2.4, R2.1; no longer IC5.4, R4.1
- net 6: now also JP4.3; no longer JP8.3
- net 7: now also JP4.1; no longer JP8.1
- net A0: now also JP1.1; no longer JP4.1
- net GND: now also C1.2, C12.2, C14.2, C15.2, C16.2, C2.2, IC1.2, IC1.5, IC3.2, IC3.5, IC4.2, IC4.5, X1.GND@0, X1.GND@1, X1.GND@2, X1.GND@3; no longer C13.2, IC5.2, IC5.5, IC6.2, IC6.5, IC7.2, IC7.5, X2.GND@2, X2.GND@3, X3.GND@0, X3.GND@1
- net GPIO1: now also IC4.4; no longer IC7.4
- net GPS_RX1: now also IC2.3; no longer IC5.3
- net GPS_TX1: now also IC3.4; no longer IC6.4
- net N$4: now also C13.2, X1.SIG, X2.SIGNAL; no longer C12.2, X2.SIG, X3.SIGNAL
- net N$5: now also IC3.3, R3.2; no longer IC6.3, R5.2
- net N$7: now also C13.1; no longer C12.1
- net N$8: now also IC1.4, JP1.2; no longer IC2.4, JP4.2
- net PPS: now also IC4.3, JP4.2; no longer IC7.3, JP8.2
- net V_ANT: now also C14.1, C15.1, C16.1, JP2.2; no longer C13.1, JP6.2
Routing:
- net IOREF: track 0.62 -> 0.00 mm
- net N$8: track 0.62 -> 0.00 mm
Other:
- board outline removed
- board text removed: "Arduino NV08C GPS Shield v1.0"
- board text removed: "Steve Marple Lancaster University"
