File: hardware/NV08C_GPS_shield_v1.1_reduced.sch (EAGLE design)
At the start: 36 parts, among them IC2 74LVC1T45SOT23-HAND, IC5 74LVC1T45SOT23-HAND, IC6 74LVC1T45SOT23-HAND, IC7 74LVC1T45SOT23-HAND, X2 CONN-SMATHD, X3 UFL

Commit message: Layout fixes
Parts:
- removed IC5: 74LVC1T45SOT23-HAND, SteveMarple:74LVC1T45SOT23-HAND
- removed JP6: V ANT, SparkFun:JUMPER-3PTH
- removed JP8: PPS 7/6, SparkFun:JUMPER-3PTH
- removed X3: UFL, SteveMarple:CONN-UFLHAND
- added C1, C2: 100n, SteveMarple:C-EU1206-HAND
- added C14: 22p, SteveMarple:C-EU0805-HAND
- added C15: 1u, SteveMarple:C-EU1206-HAND
- added C16: 4u7, SteveMarple:CAP_POLPTH2
- added IC1: 74LVC1T45SOT23-HAND, SteveMarple:74LVC1T45SOT23-HAND
- added JP1: GPS !RESET! (A0), SparkFun:JUMPER-2PTH
- added JP2: V ANT, SparkFun:JUMPER-3PTH
- added X1: CONN-SMATHD, SteveMarple:CONN-SMATHD
- C10: value 1u -> 22p; device SteveMarple:C-EU1206-HAND -> SteveMarple:C-EU0805-HAND
- C12, C9: value 22p -> 1u; device SteveMarple:C-EU0805-HAND -> SteveMarple:C-EU1206-HAND
- C7, C8: value 1u -> 100n
- JP4: value GPS !RESET! (A0) -> PPS 7/6; device SparkFun:JUMPER-2PTH -> SparkFun:JUMPER-3PTH
- X2: value CONN-SMATHD -> UFL; device SteveMarple:CONN-SMATHD -> SteveMarple:CONN-UFLHAND
- renumbered IC6 to IC3, IC7 to IC4, JP7 to JP3, R4 to R2, R5 to R3, U$16 to U$1, U$18 to U$2, U$19 to U$3, U$20 to U$4, U$21 to U$5, U$22 to U$6, U$23 to U$7, U$24 to U$8, U$25 to U$9
Connections:
- removed net IOREF: C3.1, C4.1, IC2.VCC_B, IC3.VCC_A, IC4.VCC_A, IC5.VCC_B, R1.2, R2.2
- new net VCC: C1.1, C2.1, C3.1, C4.1, IC1.VCC_B, IC2.VCC_B, IC3.VCC_A, IC4.VCC_A, R1.2, R2.2
- net !GPS_RESET: now also IC1.A; no longer IC2.A
- net +3V3: now also C12.1, C7.1, IC1.VCC_A, JP2.3; no longer IC5.VCC_A, JP6.3
- net +5V: now also JP2.1; no longer C7.1, JP6.1
- net 3(TX1): now also IC2.B; no longer IC5.B
- net 6: now also JP4.3; no longer JP8.3
- net 7: now also JP4.1; no longer JP8.1
- net A0: now also JP1.1; no longer JP4.1
- net GND: now also C1.2, C12.2, C14.2, C15.2, C16.-, C2.2, IC1.DIR, IC1.GND, X1.GND; no longer C13.2, IC5.DIR, IC5.GND, X3.GND
- net GPS_RX1: now also IC2.A; no longer IC5.A
- net N$4: now also C13.2, X1.SIGNAL; no longer C12.2, X3.SIGNAL
- net N$7: now also C13.1; no longer C12.1
- net N$8: now also IC1.B, JP1.2; no longer IC2.B, JP4.2
- net PPS: now also JP4.2; no longer JP8.2
- net V_ANT: now also C14.1, C15.1, C16.+, JP2.2; no longer C13.1, JP6.2
Other:
- note added: "74LVC1T45 decoupling"
- moved on the sheet: C10, C11, C12, C13, C3, C4, C5, C6, C7, C8, C9, IC2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
