File: hardware/Calunium_v2_smd_2.brd (EAGLE design)
At the start: 99.1 x 78.7 mm, 64 parts, among them IC1 LD1117S33TR, IC2 DS1338, IC4 ATMEGA1284, IC5 MCP2200, IC6 TSR 1-2450, Q1 2N7002, X1 PWR, X2 JTAG, X3 USB, X6 MICRO-SD-SOCKETHIROSE-DM3D, Y1 32k768, Y2 16MHz, Y3 12MHz

Commit message: Add schematics and boards for various modules
Parts:
- Q1: value 2N7002 -> BSS138; device SteveMarple:SOT23-3-ROTATED -> SteveMarple:SOT23-3-HAND
Changed lines of the file:
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@@
 <attribute name="VALUE" x="72.39" y="1.27" size="1.27" layer="27"/>
 </element>
-<element name="Q1" library="SteveMarple" package="SOT23-3-ROTATED" value="2N7002" x="12.7" y="72.39" smashed="yes" rot="R270">
+<element name="Q1" library="SteveMarple" package="SOT23-3-HAND" value="BSS138" x="12.7" y="72.39" smashed="yes" rot="R270">
 <attribute name="NAME" x="9.2075" y="69.85" size="1.27" layer="25" ratio="10" rot="R90"/>
 <attribute name="VALUE" x="10.795" y="69.85" size="1.27" layer="27" ratio="10" rot="R90"/>
-<attribute name="PACKAGE" value="SOT-23-3" x="12.7" y="72.39" size="1.778" layer="27" rot="R270" display="off"/>
-<attribute name="OC_NEWARK" value="25R5679" x="12.7" y="72.39" size="1.778" layer="27" rot="R270" display="off"/>
-<attribute name="MPN" value="2N7002-7-F" x="12.7" y="72.39" size="1.778" layer="27" rot="R270" display="off"/>
-<attribute name="SUPPLIER" value="DIODES INC." x="12.7" y="72.39" size="1.778" layer="27" rot="R270" display="off"/>
-<attribute name="OC_FARNELL" value="1713823" x="12.7" y="72.39" size="1.778" layer="27" rot="R270" display="off"/>
 </element>
 <element name="IC2" library="SteveMarple" package="SO08" value="DS1338" x="90.17" y="20.32" smashed="yes">
@@
 <wire x1="18.46" y1="62.865" x2="22.86" y2="66.675" width="0" layer="19" extent="1-1"/>
 <wire x1="26.416" y1="76.2" x2="22.86" y2="66.675" width="0" layer="19" extent="1-1"/>
-<wire x1="11.684" y1="73.406" x2="18.46" y2="62.865" width="0" layer="19" extent="1-1"/>
-<wire x1="11.201" y1="76.2" x2="11.684" y2="73.406" width="0" layer="19" extent="1-1"/>
+<wire x1="11.684" y1="74.041" x2="18.46" y2="62.865" width="0" layer="19" extent="1-1"/>
+<wire x1="11.201" y1="76.2" x2="11.684" y2="74.041" width="0" layer="19" extent="1-1"/>
 <wire x1="4.445" y1="74.295" x2="11.201" y2="76.2" width="0" layer="19" extent="1-1"/>
 </signal>
@@
 <contactref element="LED1" pad="K"/>
 <contactref element="Q1" pad="3"/>
-<wire x1="3.81" y1="21.59" x2="12.7" y2="71.374" width="0" layer="19" extent="1-1"/>
+<wire x1="3.81" y1="21.59" x2="12.7" y2="70.739" width="0" layer="19" extent="1-1"/>
 </signal>
 <signal name="13(SCK)">
@@
 <wire x1="28.956" y1="76.2" x2="35.56" y2="59.69" width="0" layer="19" extent="1-1"/>
 <wire x1="14.199" y1="76.2" x2="28.956" y2="76.2" width="0" layer="19" extent="1-1"/>
-<wire x1="13.716" y1="73.406" x2="14.199" y2="76.2" width="0" layer="19" extent="1-1"/>
+<wire x1="13.716" y1="74.041" x2="14.199" y2="76.2" width="0" layer="19" extent="1-1"/>
 </signal>
 <signal name="VBATT">
