File: hardware/Calunium_v2_smd_2.sch (EAGLE design)
At the start: 67 parts, among them IC1 MCP1702-3.3, IC2 DS1338, IC3 MCP1702-5.0, IC4 ATMEGA1284, IC5 MCP2200, Q1 2N7000, X1 PWR, X2 JTAG, X3 USB, X4 CONN-SMATHD, X5 UART0, X6 MICRO-SD-SOCKETHIROSE-DM3D, Y1 32k768, Y2 16MHz, Y3 12MHz

Commit message: Misc changes
Parts:
- removed F1: PTCPTH, SparkFun:PTCPTH
- removed IC3: MCP1702-5.0, SteveMarple:MCP1702
- removed JP4: D6 SQW/RFM12B, SparkFun:JUMPER-3PTH
- removed JP6: VREG PWR, SparkFun:JUMPER-2PTH
- removed RF1: RFM12B, SteveMarple:RFM12BSMD
- removed X4: CONN-SMATHD, SteveMarple:CONN-SMATHD
- removed X5: UART0, SparkFun:ARDUINO_SERIAL_PROGRAMPTH
- added C19, C20: 100n, SteveMarple:C-EU1206-HAND
- added IC6: TSR 1-2450, SteveMarple:V_REG_78XXTSR-1-XXXX
- added L2: FERRITE, SteveMarple:INDUCTOR0805-HAND
- C1, C8: device SparkFun:CAPPTH1 -> SteveMarple:C-EU1206-HAND
- C10, C11, C15, C16, C17, C18: device SparkFun:CAPPTH -> SteveMarple:C-EU0805-HAND
- C12, C14, C3, C4, C5, C7, C9: device SparkFun:CAPPTH -> SteveMarple:C-EU1206-HAND
- C13: value 100n -> 10n; device SparkFun:CAPPTH -> SteveMarple:C-EU1206-HAND
- C2: value 1u -> 10u; device SparkFun:CAPPTH1 -> SteveMarple:CAP_POLPTH2
- D1, D2: device SteveMarple:DIODE-SCHOTTKY -> SteveMarple:DIODE-SCHOTTKYSOT23-1-3-HAND
- IC1: value MCP1702-3.3 -> LD1117S33TR; device SteveMarple:MCP1702 -> SteveMarple:V_REG_LD1117VXXSOT223-HAND
- JP1: value SQW D15 -> SQW D6/D15; device SparkFun:JUMPER-2PTH -> SparkFun:JUMPER-3PTH
- JP9: value USB/FTDI -> USB/VIN
- L1: device SteveMarple:INDUCTOR0.4"-AXIAL -> SteveMarple:INDUCTOR1210-HAND
- Q1: value 2N7000 -> 2N7002; device SteveMarple:2N7000 -> SteveMarple:2N7002
- R1, R2: value 1k -> 560R; device SteveMarple:RESISTOR -> SteveMarple:RESISTOR1206-HAND
- R10, R3, R4, R5, R6, R7, R9: device SteveMarple:RESISTOR -> SteveMarple:RESISTOR1206-HAND
- R8: value 100k -> 0R; device SteveMarple:RESISTOR -> SteveMarple:RESISTOR1206-HAND
Connections:
- net N$21 renamed !MCP2200_RESET
- removed net N$10: JP9.1, X5.VCC
- removed net N$17: RF1.ANT, X4.SIGNAL
- removed net RFM12B_!IRQ: JP4.3, RF1.!IRQ
- net +3V3: now also C19.1, C2.+, IC1.OUT; no longer C2.1, IC1.VOUT
- net +5V: now also IC1.IN, JP9.2; no longer F1.2, IC1.VIN, JP6.2
- net +5V_USB: now also C13.1, JP9.3, L2.2; no longer F1.1, JP9.2
- net 0(RX0): no longer X5.TXO
- net 1(TX0): no longer X5.RXI
- net 11(MOSI): no longer RF1.SDI
- net 12(MISO): no longer RF1.SDO
- net 13(SCK): no longer RF1.SCK
- net 14: no longer R8.1, RF1.!SEL
- net 6: now also JP1.3; no longer JP4.2
- net AUTO_RESET: no longer X5.DTR
- net GND: now also C19.2, C2.-, C20.2, IC6.GND; no longer C2.2, IC3.GND, RF1.GND, X4.GND, X5.GND
- net N$11: now also R8.2
- net N$14: now also IC6.OUT, JP9.1; no longer IC3.VOUT, JP6.1
- net N$16: now also L2.1; no longer JP9.3
- net SQW: no longer JP4.1
- net VBATT: now also R8.1
- net VCC: now also C20.1; no longer C13.1, R8.2, RF1.VDD
- net VIN: now also IC6.IN; no longer IC3.VIN
Other:
- note added: "TODO Swap MCP1702 (3V3 and 5V) for SMD"
- note added: "USB power and filtering"
- note removed: "FTDI for UART0"
- note removed: "Pull-up disables RFM12B"
- note removed: "RFM12B radio module"
- note removed: "when ICSP in use"
- moved on the sheet: C12, C13, D2, H1, H2, H3, H4, JP7, JP9, R7, R8, R9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

Commit message: Add schematics and boards for various modules
Parts:
- Q1: value 2N7002 -> BSS138; device SteveMarple:2N7002 -> SteveMarple:BSS138SOT23-3-HAND
Changed lines of the file:
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@@
 <part name="FRAME1" library="SteveMarple" deviceset="FRAME-A3" device=""/>
 <part name="X3" library="SteveMarple" deviceset="USB" device="PTH" value="USB"/>
-<part name="Q1" library="SteveMarple" deviceset="2N7002" device=""/>
+<part name="Q1" library="SteveMarple" deviceset="BSS138" device="SOT23-3-HAND" value="BSS138"/>
 <part name="IC2" library="SteveMarple" deviceset="DS1307" device="SO08" value="DS1338"/>
 <part name="LED1" library="SparkFun" deviceset="LED" device="3MM" value="D13"/>
@@
 <instance part="FRAME1" gate="G$1" x="-172.72" y="-76.2"/>
 <instance part="X3" gate="G$1" x="-144.78" y="-20.32" smashed="yes" rot="MR0"/>
-<instance part="Q1" gate="A" x="185.42" y="132.08"/>
+<instance part="Q1" gate="G$1" x="185.42" y="132.08"/>
 <instance part="IC2" gate="G$1" x="142.24" y="66.04"/>
 <instance part="LED1" gate="G$1" x="185.42" y="142.24"/>
@@
 </segment>
 <segment>
-<pinref part="Q1" gate="A" pin="S"/>
+<pinref part="Q1" gate="G$1" pin="S"/>
 <pinref part="GND3" gate="1" pin="GND"/>
 <wire x1="185.42" y1="127" x2="185.42" y2="119.38" width="0.1524" layer="91"/>
@@
 <segment>
 <pinref part="LED1" gate="G$1" pin="C"/>
-<pinref part="Q1" gate="A" pin="D"/>
+<pinref part="Q1" gate="G$1" pin="D"/>
 </segment>
 </net>
@@
 </segment>
 <segment>
-<pinref part="Q1" gate="A" pin="G"/>
+<pinref part="Q1" gate="G$1" pin="G"/>
 <wire x1="180.34" y1="129.54" x2="172.72" y2="129.54" width="0.1524" layer="91"/>
 <label x="165.1" y="129.54" size="1.778" layer="95" rot="MR0"/>
